File: PAL V2/PCB pal/PCB pal.kicad_pcb (KiCad board)
At the start: 2 copper layers, 35.2 x 83.7 mm, 8 parts, among them J1 Conn_01x04_MountingPin, J2 Conn_01x02, M1 Motor_Servo, M2 Motor_Servo, M3 Motor_Servo, M4 Motor_Servo, P1 USB_C_Plug_USB2.0, U1 ESP32-C6-DEVKITC-1-N8

Commit message: New PCB changes
Parts:
- removed M3, M4: Motor_Servo, Connector_PinHeader_1.00mm:PinHeader_1x03_P1.00mm_Horizontal
- removed P1: USB_C_Plug_USB2.0, USBC:GCT_USB4140-GF-0070-C_REVA3
- added ?: LOGO, faces:fuck, F.Cu at (33.8, 49.3)
- added G***: LOGO, faces:fuck, B.Cu at (31.2, 51.5)
- added J3: Conn_01x02, modified:BatteryTERMINAL, F.Cu at (49.7, 18.4)
- J1: footprint Connector_PinHeader_1.00mm:PinHeader_1x04_P1.00mm_Horizontal -> Connector_PinHeader_2.00mm:PinHeader_1x04_P2.00mm_Vertical
- J2: footprint Connector_PinHeader_1.00mm:PinHeader_1x02_P1.00mm_Horizontal -> Connector_PinHeader_2.00mm:PinHeader_1x02_P2.00mm_Vertical
- M1, M2: footprint Connector_PinHeader_1.00mm:PinHeader_1x03_P1.00mm_Horizontal -> Connector_PinHeader_2.00mm:PinHeader_1x03_P2.00mm_Vertical
- moved J2 96.3 mm to (53.0, 23.9), turned to 0 degrees
- moved U1 42.9 mm to (31.8, 44.1), turned to 180 degrees
- moved M1 42.7 mm to (53.1, 29.8), turned to 0 degrees
- moved M2 33.1 mm to (53.0, 38.8), turned to 0 degrees
- moved J1 12.3 mm to (53.1, 46.9), turned to 0 degrees
Connections:
- U1 pad J3_10: /SERVO4 -> unconnected-(U1-GPIO18-PadJ3_10)
- U1 pad J3_9: /SERVO3 -> unconnected-(U1-GPIO19-PadJ3_9)
Routing:
- net GND: track 130.5 -> 44.1 mm, vias 0 -> 1
- net /SERVO3: track 40.1 -> 0.00 mm, vias 1 -> 0
- net /SERVO4: track 39.9 -> 0.00 mm, vias 1 -> 0
- net +5V: track 53.8 -> 28.0 mm, vias 1 -> 0
- net /SDA: track 24.3 -> 35.0 mm
- net /SCL: track 27.3 -> 34.7 mm
- net +3.3V: track 32.3 -> 26.4 mm
- net Net-(J2-Pin_1): track 10.7 -> 6.26 mm
- net /SERVO2: track 40.0 -> 37.5 mm, vias 1 -> 0
- net /SERVO1: track 40.2 -> 42.4 mm
Other:
- board size 35.2 x 83.7 mm -> 50 x 70 mm
- board text added: "Luklab63"

Commit message: shoulder mount
Parts:
- moved J1 110.2 mm to (148.9, 101.3)
- moved J3 110.2 mm to (145.5, 72.8)
- moved M1 110.2 mm to (148.9, 84.2)
- moved M2 110.2 mm to (148.8, 93.2)
- moved ? 110.2 mm to (129.6, 103.7)
- moved G*** 110.2 mm to (127.0, 105.9)
- moved U1 110.2 mm to (127.6, 98.5)
- moved J2 110.2 mm to (148.8, 78.3)
Other:
- outline, holes or cut-outs redrawn

Commit message: ESP BOX+ PCB
Parts:
- removed the G*** at (127.0, 105.9)
- added ?: LOGO, faces:NOAI, B.Cu at (23.3, 36.7)
- added G***: LOGO, faces:piment, F.Cu at (41.9, 60.5)
- added G***: LOGO, faces:NOAI smol, F.Cu at (44.5, 47.8)
- moved J1 126.6 mm to (41.1, 34.9)
- moved J3 126.6 mm to (37.7, 6.40)
- moved M1 126.6 mm to (41.1, 17.8)
- moved M2 126.6 mm to (41.0, 26.8)
- moved ? 126.6 mm to (21.8, 37.3)
- moved J2 126.6 mm to (41.0, 11.9)
- moved U1 126.6 mm to (19.8, 32.1)
Routing:
- net GND: track 44.1 -> 53.8 mm
- net +3.3V: track 26.4 -> 16.7 mm
Other:
- outline, holes or cut-outs redrawn
- board text added: "Made on earth by a human"

Commit message: PCB finished and sent to print
Parts:
- removed the ? at (23.3, 36.7)
- added D1: LED, LED_THT:LED_D3.0mm, F.Cu at (46.3, 9.00)
- added D2: LED, LED_THT:LED_D3.0mm, F.Cu at (46.2, 42.1)
- added R 220: R 220, Resistor_THT:R_Axial_DIN0207_L6.3mm_D2.5mm_P10.16mm_Horizontal, F.Cu at (46.3, 14.4)
- added R 220: R 220, Resistor_THT:R_Axial_DIN0207_L6.3mm_D2.5mm_P10.16mm_Horizontal, F.Cu at (46.3, 36.9)
- moved G*** 3.21 mm to (41.3, 47.5)
- moved ? 2.70 mm to (21.1, 34.7)
- moved G*** 2.30 mm to (40.6, 58.6)
Routing:
- net GND: track 53.8 -> 3.14 mm
- net +3.3V: track 16.7 -> 26.4 mm
- net +5V: track 28.0 -> 37.3 mm
- net Net-(D1-A): track 0.00 -> 2.88 mm
- net Net-(D2-A): track 0.00 -> 2.69 mm
- net /SERVO2: vias 0 -> 2
- added copper zone on B.Cu, net GND
Other:
- outline, holes or cut-outs redrawn

Commit message: PCB EDIT + STEP FILES
Parts:
- J1: footprint Connector_PinHeader_2.00mm:PinHeader_1x04_P2.00mm_Vertical -> Connector_PinHeader_2.54mm:PinHeader_1x04_P2.54mm_Vertical
- J2: footprint Connector_PinHeader_2.00mm:PinHeader_1x02_P2.00mm_Vertical -> Connector_PinHeader_2.54mm:PinHeader_1x02_P2.54mm_Vertical
- M1, M2: footprint Connector_PinHeader_2.00mm:PinHeader_1x03_P2.00mm_Vertical -> Connector_PinHeader_2.54mm:PinHeader_1x03_P2.54mm_Vertical
- R1, R2: renamed from R 220; value R 220 -> R
- moved M1 4.00 mm to (41.3, 13.8)
- moved J2 3.84 mm to (37.3, 13.0)
- moved M2 2.30 mm to (41.1, 24.5)
- moved J1 0.24 mm to (41.0, 34.7)
Routing:
- net /SERVO1: track 42.4 -> 44.3 mm
- net Net-(J2-Pin_1): track 6.26 -> 7.37 mm
- net /SERVO2: track 37.5 -> 38.6 mm
- net /SDA: track 35.0 -> 34.3 mm
Other:
- outline, holes or cut-outs redrawn
